Commit message: Stefano:renamed ur robots

File: ur_description/urdf/ur.gazebo.xacro (robot description, xacro)
@@ -2,25 +2,5 @@
 <robot xmlns:xacro="http://ros.org/wiki/xacro">
   <xacro:macro name="ur_arm_gazebo" params="prefix">
-    <gazebo reference="${prefix}shoulder_link">
-      <selfCollide>true</selfCollide>
-    </gazebo>
-    <gazebo reference="${prefix}upper_arm_link">
-      <selfCollide>true</selfCollide>
-    </gazebo>
-    <gazebo reference="${prefix}forearm_link">
-      <selfCollide>true</selfCollide>
-    </gazebo>
-    <gazebo reference="${prefix}wrist_1_link">
-      <selfCollide>true</selfCollide>
-    </gazebo>
-    <gazebo reference="${prefix}wrist_3_link">
-      <selfCollide>true</selfCollide>
-    </gazebo>
-    <gazebo reference="${prefix}wrist_2_link">
-      <selfCollide>true</selfCollide>
-    </gazebo>
-    <gazebo reference="${prefix}ee_link">
-      <selfCollide>true</selfCollide>
-    </gazebo>
+    <!-- nothing to do here at the moment -->
   </xacro:macro>
 </robot>

File: ur_description/urdf/ur5_joint_limited_robot.urdf.xacro (robot description, xacro)
@@ -7,5 +7,5 @@
   <xacro:include filename="$(find ur_description)/urdf/ur5.urdf.xacro" />
   <!-- arm -->
-  <xacro:ur5_robot prefix="" joint_limited="true"
+  <xacro:ur5_robot prefix="ur5_" joint_limited="true"
     shoulder_pan_lower_limit="${-pi}" shoulder_pan_upper_limit="${pi}"
     shoulder_lift_lower_limit="${-pi}" shoulder_lift_upper_limit="${pi}"
@@ -16,8 +16,16 @@
   />
   <link name="world" />
-  <joint name="world_joint" type="fixed">
+<!--  World joints of ur5-->
+  <joint name="ur5" type="fixed">
     <parent link="world" />
-    <child link = "base_link" />
+    <child link = "ur5_base_link" />
     <origin xyz="0.0 0.0 0.0" rpy="0.0 0.0 0.0" />
   </joint>
+<!--  World joints of ur10-->
+<!--  <link name="ur10" />
+  <joint name="ur10_world_joint" type="fixed">
+    <parent link="world" />
+    <child link = "ur10_base_link" />
+    <origin xyz="0.0 0.0 0.0" rpy="0.0 0.0 0.0" />
+  </joint>-->
 </robot>
