Commit message: manue

File: ur_description/urdf/ur10.urdf.xacro (robot description, xacro)
@@ -14,5 +14,5 @@
   <xacro:property name="wrist_1_mass" value="1.96" />
   <xacro:property name="wrist_2_mass" value="1.96" />
-  <xacro:property name="wrist_3_mass" value="0.202" />
+  <xacro:property name="wrist_3_mass" value="1"  /> <!--"0.202"-->
   <!-- These parameters are borrowed from the urcontrol.conf file
        but are not verified for the correct permutation.
